File: E7009E_blameless_project.kicad_pcb (KiCad board)
At the start: 2 copper layers, 70.3 x 57.5 mm, 74 parts, among them M1 IRF9530, P1 CONN_01X06, P2 CONN_01X01, P3 CONN_01X01, P4 CONN_01X01, P5 CONN_01X01, Q1 BC556, Q10 BC546, Q11 BD135, Q12 BD136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

Commit message: Complete Circuitry and PCB design
Parts:
- moved P5 180.4 mm to (61.6, 167.0)
- moved P2 126.8 mm to (64.4, 47.0)
- moved Q10 78.4 mm to (131.1, 116.8)
- moved R18 72.7 mm to (129.7, 123.8), turned to 180 degrees
- moved P4 62.3 mm to (248.4, 142.1)
- moved C5 54.5 mm to (142.1, 90.7)
- moved R1 45.6 mm to (143.4, 77.2), turned to 0 degrees
- moved R4 33.8 mm to (155.7, 68.9), turned to 0 degrees
- moved R5 26.1 mm to (164.9, 75.7), turned to 0 degrees
- moved Q6 17.1 mm to (173.4, 83.7)
- moved C6 9.21 mm to (184.6, 71.3)
- moved Q4 5.89 mm to (189.9, 100.9)
- moved Q1 5.89 mm to (185.6, 97.8)
- moved Q2 5.89 mm to (185.6, 103.4)
- moved Q5 5.89 mm to (190.7, 97.8)
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Routing:
- net GNDPWR: track 349.4 -> 3.11 mm, vias 69 -> 0
- net GND: track 189.7 -> 10.2 mm, vias 40 -> 0
- net /VSS: track 198.3 -> 114.0 mm
- net Net-(Q5-Pad2): track 52.1 -> 11.5 mm
- net Net-(C5-Pad1): track 28.9 -> 0.00 mm
- net Net-(Q10-Pad2): track 25.0 -> 0.00 mm
- net /VDD: track 108.9 -> 87.1 mm
- net /VAS: track 42.0 -> 21.6 mm
- net Net-(Q3-Pad3): track 19.4 -> 0.00 mm
- net Net-(Q3-Pad2): track 18.6 -> 5.97 mm
- net Net-(Q6-Pad2): track 7.88 -> 0.00 mm
- net Net-(C10-Pad2): track 39.8 -> 36.5 mm
- net Net-(C8-Pad2): track 7.75 -> 10.4 mm
- net Net-(C11-Pad1): track 34.3 -> 32.6 mm
- net Net-(Q5-Pad3): track 5.45 -> 3.80 mm
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Other:
- board outline removed
