File: Kicad/E7009E_blameless_project.sch (KiCad schematic (older format))
At the start: 66 parts, among them M5 IRF9530, M7 IRF9530, P1 CONN_01X06, Q1 BC556, Q15 BD135, Q16 BD135, Q17 BD136, Q18 BC556, Q19 BC556, Q2 BC556, Q3 BC556, Q5 BC546, Q6 BC546, Q8 BC546, Q9 BC546

Commit message: Complete Circuitry and PCB design
Parts:
- removed M7: IRF9530, symbol IRF9530
- added C11: 1n, Capacitors_ThroughHole:C_Disc_D3.0mm_W1.6mm_P2.50mm, symbol C
- added P2, P3, P4, P5: CONN_01X01, Custom_Holes:Mounting_D3mm_Pad1mm_totd6mm, symbol CONN_01X01
- added Q13: IRF530, TO_SOT_Packages_THT:TO-220_Vertical, symbol IRF530
- added R36, R37, R38: 100, Resistors_ThroughHole:R_Axial_DIN0204_L3.6mm_D1.6mm_P5.08mm_Horizontal, symbol R
- C1, C2: footprint Capacitors_THT:C_Disc_D3.0mm_W1.6mm_P2.50mm -> Capacitors_ThroughHole:C_Disc_D3.0mm_W2.0mm_P2.50mm
- C10: renamed from C8; footprint (none) -> Capacitors_ThroughHole:CP_Radial_D5.0mm_P2.50mm; symbol C -> CP
- C12: renamed from C9; value 2.2n -> 1n; footprint (none) -> Capacitors_ThroughHole:C_Disc_D3.0mm_W1.6mm_P2.50mm
- C13: footprint (none) -> Capacitors_ThroughHole:C_Disc_D3.0mm_W2.0mm_P2.50mm; symbol CP -> C
- C14: renamed from C15; footprint (none) -> Capacitors_ThroughHole:C_Disc_D3.0mm_W2.0mm_P2.50mm
- C15: renamed from C14; footprint (none) -> Capacitors_ThroughHole:C_Disc_D3.0mm_W2.0mm_P2.50mm
- C3, C4: footprint Capacitors_THT:CP_Radial_Tantal_D4.5mm_P5.00mm -> Capacitors_ThroughHole:CP_Radial_D8.0mm_P5.00mm
- C5: renamed from C17; footprint (none) -> Capacitors_ThroughHole:C_Disc_D3.0mm_W2.0mm_P2.50mm
- C6: renamed from C21; footprint (none) -> Capacitors_ThroughHole:C_Disc_D3.0mm_W2.0mm_P2.50mm
- C7: footprint (none) -> Capacitors_ThroughHole:CP_Radial_D8.0mm_P5.00mm
- C8: renamed from C19; footprint (none) -> Capacitors_ThroughHole:CP_Radial_D5.0mm_P2.50mm
- C9: renamed from C6; footprint (none) -> Capacitors_ThroughHole:C_Disc_D3.0mm_W1.6mm_P2.50mm
- D1: footprint (none) -> Diodes_ThroughHole:D_5W_P5.08mm_Vertical_AnodeUp
- L1: footprint (none) -> Custom_Footprints:Coil_p11mm_L15mm_d10mm
- M1: renamed from M5; footprint (none) -> TO_SOT_Packages_THT:TO-220_Vertical
- Q11: renamed from Q16; footprint Power_transsistors:TO-220_Vertical -> TO_SOT_Packages_THT:TO-126_Vertical
- Q12: renamed from Q17; footprint Power_transsistors:TO-220_Vertical -> TO_SOT_Packages_THT:TO-126_Vertical
- Q9: renamed from Q15; footprint TO_SOT_Packages_THT:TO-220_Horizontal_Reversed -> TO_SOT_Packages_THT:TO-126_Vertical
- R1, R10, R18: footprint (none) -> Resistors_ThroughHole:R_Axial_DIN0204_L3.6mm_D1.6mm_P5.08mm_Horizontal
- R11: renamed from R38; footprint (none) -> Resistors_ThroughHole:R_Axial_DIN0204_L3.6mm_D1.6mm_P5.08mm_Horizontal
- R12: renamed from R39; footprint (none) -> Resistors_ThroughHole:R_Axial_DIN0204_L3.6mm_D1.6mm_P5.08mm_Horizontal
- R13: renamed from R12; footprint (none) -> Resistors_ThroughHole:R_Axial_DIN0204_L3.6mm_D1.6mm_P5.08mm_Horizontal
- R14: renamed from R9; footprint (none) -> Resistors_ThroughHole:R_Axial_DIN0204_L3.6mm_D1.6mm_P5.08mm_Horizontal
- R15: renamed from R13; footprint (none) -> Resistors_ThroughHole:R_Axial_DIN0204_L3.6mm_D1.6mm_P5.08mm_Horizontal
- R16: renamed from R20; footprint (none) -> Resistors_ThroughHole:R_Axial_DIN0204_L3.6mm_D1.6mm_P5.08mm_Horizontal
- R17: renamed from R44; footprint (none) -> Potentiometers:Potentiometer_Trimmer_Bourns_3296W
- R19: renamed from R15; footprint (none) -> Resistors_ThroughHole:R_Axial_DIN0204_L3.6mm_D1.6mm_P5.08mm_Horizontal
- R2: renamed from R4; footprint (none) -> Resistors_ThroughHole:R_Axial_DIN0204_L3.6mm_D1.6mm_P5.08mm_Horizontal
- R20: renamed from R16; footprint (none) -> Resistors_ThroughHole:R_Axial_DIN0204_L3.6mm_D1.6mm_P5.08mm_Horizontal
- R21: renamed from R14; footprint (none) -> Resistors_ThroughHole:R_Axial_DIN0204_L3.6mm_D1.6mm_P5.08mm_Horizontal
- R22: renamed from R21; footprint (none) -> Resistors_ThroughHole:R_Axial_DIN0204_L3.6mm_D1.6mm_P5.08mm_Horizontal
- R23: renamed from R42; footprint (none) -> Resistors_ThroughHole:R_Axial_DIN0204_L3.6mm_D1.6mm_P5.08mm_Horizontal
- R24: renamed from R43; footprint (none) -> Resistors_ThroughHole:R_Axial_DIN0204_L3.6mm_D1.6mm_P5.08mm_Horizontal
- R25: renamed from R26; footprint (none) -> Resistors_ThroughHole:R_Axial_DIN0204_L3.6mm_D1.6mm_P5.08mm_Horizontal
- R26: renamed from R25; footprint (none) -> Resistors_ThroughHole:R_Axial_DIN0204_L3.6mm_D1.6mm_P5.08mm_Horizontal
- R27: renamed from R22; footprint (none) -> Resistors_ThroughHole:R_Axial_DIN0204_L3.6mm_D1.6mm_P5.08mm_Horizontal
- R28: renamed from R41; footprint (none) -> Resistors_ThroughHole:R_Axial_DIN0204_L3.6mm_D1.6mm_P5.08mm_Horizontal
- R29: renamed from R40; footprint (none) -> Resistors_ThroughHole:R_Axial_DIN0204_L3.6mm_D1.6mm_P5.08mm_Horizontal
- R3: renamed from R2; footprint (none) -> Resistors_ThroughHole:R_Axial_DIN0204_L3.6mm_D1.6mm_P5.08mm_Horizontal
- R30: renamed from R23; footprint (none) -> Custom_Footprints:R_Axial_DIN0207_L6.3mm_D2.5mm_P17.15mm_Horizontal
- R31: renamed from R24; footprint (none) -> Custom_Footprints:R_Axial_DIN0207_L6.3mm_D2.5mm_P17.15mm_Horizontal
- R32: renamed from R30; footprint (none) -> Resistors_ThroughHole:R_Axial_DIN0414_L11.9mm_D4.5mm_P25.40mm_Horizontal
- R33: renamed from R29; footprint (none) -> Resistors_ThroughHole:R_Axial_DIN0414_L11.9mm_D4.5mm_P25.40mm_Horizontal
- R34: renamed from R33; footprint (none) -> Resistors_ThroughHole:R_Axial_DIN0204_L3.6mm_D1.6mm_P5.08mm_Horizontal
- R35: renamed from R32; footprint (none) -> Resistors_ThroughHole:R_Axial_DIN0204_L3.6mm_D1.6mm_P5.08mm_Horizontal
- R4: renamed from R6; footprint (none) -> Resistors_ThroughHole:R_Axial_DIN0204_L3.6mm_D1.6mm_P5.08mm_Horizontal
- R5: renamed from R31; footprint (none) -> Resistors_ThroughHole:R_Axial_DIN0204_L3.6mm_D1.6mm_P5.08mm_Horizontal
- R6: renamed from R5; footprint (none) -> Resistors_ThroughHole:R_Axial_DIN0204_L3.6mm_D1.6mm_P5.08mm_Horizontal
- R7: renamed from R3; footprint (none) -> Resistors_ThroughHole:R_Axial_DIN0204_L3.6mm_D1.6mm_P5.08mm_Horizontal
- R8: renamed from R35; footprint (none) -> Resistors_ThroughHole:R_Axial_DIN0204_L3.6mm_D1.6mm_P5.08mm_Horizontal
- R9: renamed from R36; value 400 -> 100; footprint (none) -> Resistors_ThroughHole:R_Axial_DIN0204_L3.6mm_D1.6mm_P5.08mm_Horizontal
- renumbered Q2 to Q1, Q9 to Q10, Q5 to Q2, Q1 to Q3, Q6 to Q4, Q3 to Q5, Q19 to Q6, Q18 to Q7
Connections:
- net GND: now also P1.2 (P2); no longer C13.2, P1.3 (P3), P1.4 (P4), R23.2, R24.1
- net GNDPWR: now also C13.2, P1.5 (P5), R23.2, R24.1
- net INPUT: now also P1.1 (P1); no longer P1.2 (P2)
- net OUTPUT: now also L1.1, P1.6 (P6); no longer L1.2, P1.5 (P5)
- net VAS: now also C11.2
- net VDD: now also M1.3 (S), P1.3 (P3); no longer P1.6 (P6)
- net VSS: now also P1.4 (P4), Q13.3 (S); no longer P1.1 (P1)
- net feedback: now also L1.2; no longer L1.1
- net at Q11.3 (B), Q7.1 (C), R19.2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: now also C10.1; no longer C10.2
- net at R10.1, R8.1: now also R9.1; no longer R9.2
- net at C7.1, D1.1 (K): now also R37.1; no longer R9.1
- net at Q10.1 (C), Q9.1 (E), R17.2: now also C10.2; no longer C10.1
- net at C12.1, Q12.3 (B): now also C11.1
- net at R27.2: now also M1.1 (G)
- net at R29.1, R30.2, R35.2: now also M1.2 (D)
- net at R26.2: now also Q13.1 (G)
- net at R28.2, R31.2, R34.1: now also Q13.2 (D)
- new net: R36.2, R9.2
- new net: R36.1, R38.1
- new net: R37.2, R38.2
- no-connect marks 0 -> 4
Other:
- moved on the sheet: C1, C2, C3, C4, L1, M1, R9
