File: Kicad/_autosave-E7009E_blameless_project.kicad_pcb (KiCad board)
At the start: 2 copper layers, 74 parts, among them M1 IRF9530, P1 CONN_01X06, P2 CONN_01X01, P3 CONN_01X01, P4 CONN_01X01, P5 CONN_01X01, Q1 BC556, Q10 BC546, Q11 BD135, Q12 BD136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

Commit message: All
Parts:
- moved P4 185.4 mm to (64.6, 117.8)
- moved P3 126.6 mm to (121.9, 74.6)
- moved C13 126.0 mm to (101.9, 103.4)
- moved C3 126.0 mm to (86.8, 78.0)
- moved C9 126.0 mm to (91.9, 113.8)
- moved M1 126.0 mm to (125.4, 87.0)
- moved Q13 126.0 mm to (125.4, 117.0)
- moved Q7 126.0 mm to (76.3, 82.1)
- moved R13 126.0 mm to (91.8, 111.0)
- moved R17 126.0 mm to (77.3, 94.8)
- moved R19 126.0 mm to (73.3, 92.9)
- moved R20 126.0 mm to (73.3, 100.1)
- moved R25 126.0 mm to (114.9, 122.1)
- moved R26 126.0 mm to (117.1, 117.1)
- moved R27 126.0 mm to (117.1, 87.1)
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Routing:
- net GNDPWR: track 3.11 -> 349.4 mm, vias 0 -> 69
- net GND: track 10.2 -> 189.7 mm, vias 0 -> 40
- net /VSS: track 106.0 -> 198.3 mm
- net Net-(Q5-Pad2): track 7.86 -> 52.4 mm
- net /VAS: track 2.50 -> 42.0 mm
- net Net-(C5-Pad1): track 0.00 -> 28.9 mm
- net Net-(Q10-Pad2): track 0.00 -> 25.0 mm
- net /VDD: track 87.1 -> 108.9 mm
- net Net-(Q3-Pad3): track 0.00 -> 19.4 mm
- net Net-(Q3-Pad2): track 0.00 -> 18.6 mm
- net /INPUT: track 0.00 -> 13.8 mm
- net Net-(Q2-Pad2): track 0.00 -> 13.3 mm
- net Net-(Q6-Pad2): track 0.00 -> 7.88 mm
- net Net-(C8-Pad2): track 0.00 -> 7.75 mm
- net Net-(Q3-Pad1): track 0.00 -> 7.19 mm
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Other:
- board outline added: 70.3 x 57.5 mm
